Commit message: Change for visualizing purposes

File: ouster_description/urdf/OS1-64.urdf.xacro (robot description, xacro)
@@ -6,31 +6,5 @@
       <xacro:insert_block name="origin" />
       <parent link="${parent}"/>
-      <child link="${name}_base_link"/>
-    </joint>
-    <link name="${name}_base_link" />
-    <joint name="${name}_base_to_baseplate" type="fixed">
-      <parent link="${name}_base_link"/>
-      <child link="${name}_baseplate" />
-      <origin xyz="0 0 0.008"/>
-    </joint>
-    <link name="${name}_baseplate">
-      <visual>
-        <geometry>
-          <box size="0.112 0.112 0.016" />
-        </geometry>
-        <material name="silver">
-          <color rgba="0.5 0.5 0.5 1.0" />
-        </material>
-      </visual>
-      <collision>
-        <geometry>
-          <box size="0.112 0.112 0.016" />
-        </geometry>
-      </collision>
-    </link>
-    <joint name="${name}_baseplate_to_body" type="fixed">
-      <parent link="${name}_baseplate"/>
       <child link="${name}"/>
-      <origin xyz="0 0 0.042" rpy="0 0 0" />
     </joint>
     <link name="${name}">
